File: Lamp Matrix Tester.kicad_sch (KiCad schematic)
At the start: 11 parts, among them J1 Columns, J2 Rows, U1 1088AS

Commit message: Migrate to Kicad 8 + Included symbol/footprint and 3D model for 1088AS module
Parts:
- U1: footprint Library:Led_1088AS_8x8_P2.54mm -> LampMatrixTesterLibrary:Led_1088AS_8x8_P2.54mm
Changed lines of the file:
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@@
       (effects (font (size 1.27 1.27)))
     )
-    (property "Footprint" "Library:Led_1088AS_8x8_P2.54mm" (at 143.51 21.59 0)
+    (property "Footprint" "LampMatrixTesterLibrary:Led_1088AS_8x8_P2.54mm" (at 143.51 21.59 0)
       (effects (font (size 1.27 1.27)) hide)
     )
