File: Lamp Matrix Tester.kicad_sch (KiCad schematic)
At the start: 11 parts, among them J1 Columns, J2 Rows, U1 1088AS

Commit message: V1.1 - Swapped rows and cols position and pinout
Other:
- company: (none) -> Broken Pipe
- title: (none) -> Lamp matrix tester
Changed lines of the file:
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@@
 	(generator_version "8.0")
 	(paper "A4")
+	(title_block
+		(title "Lamp matrix tester")
+		(date "2024-03-16")
+		(rev "1.0")
+		(company "Broken Pipe")
+	)
 	(wire
 		(pts
